File: tinyBox.sch (KiCad schematic (older format))
At the start: 15 parts, among them J1 USB_B_Micro, SW1 SW_DIP_x01, U1 ATSAMD21E15A-M, U2 AP2112K-3.3

Commit message: Add files via upload
Parts:
- removed D3: D_Schottky, Diode_SMD:D_0805_2012Metric_Pad1.15x1.40mm_HandSolder, symbol Device:D_Schottky
- J1: symbol Connector:USB_B_Micro -> tinyBox-rescue:USB_B_Micro-Connector
- U1: footprint Package_DFN_QFN:QFN-32-1EP_5x5mm_P0.5mm_EP3.6x3.6mm -> Package_QFP:TQFP-32_7x7mm_P0.8mm
- U2: symbol Regulator_Linear:AP2112K-3.3 -> tinyBox-rescue:AP2112K-3.3-Regulator_Linear
Connections:
- net labels added: D0_A4, D1_A0, D2_A1, D3_A3, D4_A2, D5_A5, D6
- net labels removed: VBAT
- wire segments 46 -> 49
- no-connect marks 22 -> 15
Other:
- moved on the sheet: D1, R1
Changed lines of the file:
@@
-$EndComp
-$Comp
-L MCU_Microchip_SAMD:ATSAMD21E15A-M U1
-U 1 1 5FACF219
-P 5850 3800
-F 0 "U1" H 6494 3846 50  0000 L CNN
-F 1 "ATSAMD21E15A-M" H 6494 3755 50  0000 L CNN
-F 2 "Package_DFN_QFN:QFN-32-1EP_5x5mm_P0.5mm_EP3.6x3.6mm" H 7200 1950 50  0001 C CNN
-F 3 "http://ww1.microchip.com/downloads/en/DeviceDoc/SAM_D21_DA1_Family_Data%20Sheet_DS40001882E.pdf" H 5850 3800 50  0001 C CNN
-	1    5850 3800
-	1    0    0    -1
 $EndComp
 $Comp
 L Device:R R1
 U 1 1 5FAD1CBC
-P 4700 3200
-F 0 "R1" V 4493 3200 50  0000 C CNN
-F 1 "1.5k" V 4584 3200 50  0000 C CNN
-F 2 "Resistor_SMD:R_0805_2012Metric_Pad1.20x1.40mm_HandSolder" V 4630 3200 50  0001 C CNN
-F 3 "~" H 4700 3200 50  0001 C CNN
-	1    4700 3200
-	0    -1   1    0
-$EndComp
-Wire Wire Line
-	4850 3200 5150 3200
+P 4800 3350
+F 0 "R1" V 4593 3350 50  0000 C CNN
+F 1 "1.5k" V 4684 3350 50  0000 C CNN
+F 2 "Resistor_SMD:R_0805_2012Metric_Pad1.20x1.40mm_HandSolder" V 4730 3350 50  0001 C CNN
+F 3 "~" H 4800 3350 50  0001 C CNN
+	1    4800 3350
+	1    0    0    1
+$EndComp
 $Comp
 L Device:LED D1
 U 1 1 5FAD3454
-P 4200 3200
-F 0 "D1" H 4193 3417 50  0000 C CNN
-F 1 "LED" H 4193 3326 50  0000 C CNN
-F 2 "LED_SMD:LED_0805_2012Metric_Pad1.15x1.40mm_HandSolder" H 4200 3200 50  0001 C CNN
-F 3 "~" H 4200 3200 50  0001 C CNN
-	1    4200 3200
-	1    0    0    -1
+P 4800 3700
+F 0 "D1" H 4793 3917 50  0000 C CNN
+F 1 "LED" H 4793 3826 50  0000 C CNN
+F 2 "LED_SMD:LED_0805_2012Metric_Pad1.15x1.40mm_HandSolder" H 4800 3700 50  0001 C CNN
+F 3 "~" H 4800 3700 50  0001 C CNN
+	1    4800 3700
+	0    -1   -1   0
 $EndComp
 $Comp
@@
 F 3 "http://www.led-color.com/upload/201506/APA102%20LED.pdf" H 4350 1925 50  0001 L TNN
 	1    4250 2300
-	1    0    0    -1
-$EndComp
-Wire Wire Line
-	5150 2200 4550 2200
-Wire Wire Line
-	4550 2300 5150 2300
-$Comp
-L Connector:USB_B_Micro J1
+	-1   0    0    -1
+$EndComp
+$Comp
+L tinyBox-rescue:USB_B_Micro-Connector J1
 U 1 1 5FAD9937
 P 4000 4600
@@
 	4300 4600 5150 4600
 $Comp
-L Regulator_Linear:AP2112K-3.3 U2
+L tinyBox-rescue:AP2112K-3.3-Regulator_Linear U2
 U 1 1 5FAE067C
 P 8550 3500
@@
 	1    8550 3500
 	1    0    0    -1
-$EndComp
-$Comp
-L Device:D_Schottky D3
-U 1 1 5FAE2C13
-P 7300 2800
-F 0 "D3" V 7346 2720 50  0000 R CNN
-F 1 "D_Schottky" V 7255 2720 50  0000 R CNN
-F 2 "Diode_SMD:D_0805_2012Metric_Pad1.15x1.40mm_HandSolder" H 7300 2800 50  0001 C CNN
-F 3 "~" H 7300 2800 50  0001 C CNN
-	1    7300 2800
-	0    -1   -1   0
 $EndComp
 $Comp
@@
 Text GLabel 4315 4400 2    50   Input ~ 0
 VBUS
-Text GLabel 7300 2500 1    50   Input ~ 0
-VBAT
 Text GLabel 7900 2500 1    50   Input ~ 0
 VBUS
@@
 Wire Wire Line
 	5550 1700 5550 1900
-Wire Wire Line
-	4550 3200 4350 3200
 $Comp
 L power:GND #PWR0102
 U 1 1 5FAEC182
-P 3750 3350
-F 0 "#PWR0102" H 3750 3100 50  0001 C CNN
-F 1 "GND" H 3755 3177 50  0000 C CNN
-F 2 "" H 3750 3350 50  0001 C CNN
-F 3 "" H 3750 3350 50  0001 C CNN
-	1    3750 3350
-	1    0    0    -1
-$EndComp
-Wire Wire Line
-	4050 3200 3750 3200
-Wire Wire Line
-	3750 3200 3750 3350
+P 4800 3950
+F 0 "#PWR0102" H 4800 3700 50  0001 C CNN
+F 1 "GND" H 4805 3777 50  0000 C CNN
+F 2 "" H 4800 3950 50  0001 C CNN
+F 3 "" H 4800 3950 50  0001 C CNN
+	1    4800 3950
+	1    0    0    -1
+$EndComp
 $Comp
 L power:GND #PWR0103
@@
 NoConn ~ 4300 4800
 Wire Wire Line
-	7300 2500 7300 2650
-Wire Wire Line
 	7900 2500 7900 2650
 Wire Wire Line
@@
 Wire Wire Line
 	8150 3500 8250 3500
-Wire Wire Line
-	7300 2950 7300 3400
-Wire Wire Line
-	7300 3400 7650 3400
 Connection ~ 8150 3400
-Connection ~ 7650 3400
 Wire Wire Line
 	7650 3400 7900 3400
@@
 	1    0    0    -1
 $EndComp
-NoConn ~ 5150 2400
-NoConn ~ 5150 2500
-NoConn ~ 5150 2600
-NoConn ~ 5150 2700
-NoConn ~ 5150 2800
-NoConn ~ 5150 2900
-NoConn ~ 5150 3000
-NoConn ~ 5150 3100
 NoConn ~ 5150 3300
 NoConn ~ 5150 3600
@@
 NoConn ~ 5150 4900
 NoConn ~ 5150 5000
+$Comp
+L MCU_Microchip_SAMD:ATSAMD21E15A-M U1
+U 1 1 5FACF219
+P 5850 3800
+F 0 "U1" H 6494 3846 50  0000 L CNN
+F 1 "ATSAMD21E15A-M" H 6494 3755 50  0000 L CNN
+F 2 "Package_QFP:TQFP-32_7x7mm_P0.8mm" H 7200 1950 50  0001 C CNN
+F 3 "http://ww1.microchip.com/downloads/en/DeviceDoc/SAM_D21_DA1_Family_Data%20Sheet_DS40001882E.pdf" H 5850 3800 50  0001 C CNN
+	1    5850 3800
+	1    0    0    -1
+$EndComp
+Text GLabel 5000 2500 0    50   Input ~ 0
+D1_A0
+Text GLabel 5000 2600 0    50   Input ~ 0
+D2_A1
+Text GLabel 5000 2400 0    50   Input ~ 0
+D0_A4
+Text GLabel 5000 2700 0    50   Input ~ 0
+D3_A3
+Text GLabel 5000 2800 0    50   Input ~ 0
+D4_A2
+Wire Wire Line
+	5150 3200 4800 3200
+Wire Wire Line
+	5000 2400 5150 2400
+Wire Wire Line
+	4550 2200 5150 2200
+Wire Wire Line
+	4550 2300 5150 2300
+Text GLabel 5000 2900 0    50   Input ~ 0
+D5_A5
+Text GLabel 5000 3000 0    50   Input ~ 0
+D6
+Wire Wire Line
+	5000 2500 5150 2500
+Wire Wire Line
+	5000 2600 5150 2600
+Wire Wire Line
+	5000 2700 5150 2700
+Wire Wire Line
+	5000 2800 5150 2800
+Wire Wire Line
+	5000 2900 5150 2900
+Wire Wire Line
+	5000 3000 5150 3000
+NoConn ~ 5150 3100
+Wire Wire Line
+	4800 3850 4800 3950
+Wire Wire Line
+	4800 3500 4800 3550
 $EndSCHEMATC

Commit message: Add files via upload
Parts:
- removed U1: ATSAMD21E15A-M, Package_QFP:TQFP-32_7x7mm_P0.8mm, symbol MCU_Microchip_SAMD:ATSAMD21E15A-M
- added U1: ATSAMD21E18A-A, Package_QFP:TQFP-32_7x7mm_P0.8mm, symbol MCU_Microchip_SAMD:ATSAMD21E18A-A
- renumbered D2 to D1, D1 to D2, D4 to D3, D5 to D4
Connections:
- net +3V3: now also U1.30 (VDDIN), U1.9 (VDDANA)
- net D0_A4: now also U1.3 (PA02)
- net D1_A0: now also U1.4 (PA03)
- net D2_A1: now also U1.5 (PA04)
- net D3_A3: now also U1.6 (PA05)
- net D4_A2: now also U1.7 (PA06)
- net D5_A5: now also U1.8 (PA07)
- net GND: now also U1.10 (GND), U1.28 (GND)
- net SWC: now also U1.31 (PA30)
- net SWD: now also U1.32 (PA31)
- net VBUS: now also J1.1 (VBUS)
- net at D1.1 (DI): now also U1.1 (PA00)
- net at R1.2: now also U1.13 (PA10)
- net at D1.2 (CI): now also U1.2 (PA01)
- net at J1.3 (D+): now also U1.23 (PA24)
- net at J1.2 (D-): now also U1.24 (PA25)
- net at SW1.2: now also U1.26 (~RESET)
- net at C1.2: now also U1.29 (VDDCORE)
- no-connect marks 15 -> 16
Other:
- moved on the sheet: C1, D1, D2, J1, R1, SW1

Commit message: Add files via upload
Parts:
- added J2: Conn_01x08, Connector_PinHeader_2.54mm:PinHeader_1x08_P2.54mm_Vertical, symbol Connector_Generic:Conn_01x08
Connections:
- net D0_A4: now also J2.3 (Pin_3)
- net D1_A0: now also J2.4 (Pin_4)
- net D2_A1: now also J2.5 (Pin_5)
- net D3_A3: now also J2.6 (Pin_6)
- net D4_A2: now also J2.7 (Pin_7)
- net D5_A5: now also J2.8 (Pin_8)
- net GND: now also J2.1 (Pin_1)
- new net 3V3: J2.2 (Pin_2)
Other:
- note added: "11/22/2020"
- note added: "ATSAMD21E18BA-A based clone of adafruit's trinket m0, designed for EE101"
- note added: "tinyb0x"
- moved on the sheet: R2
Changed lines of the file:
@@
 L Device:R R2
 U 1 1 5FAE6F9E
-P 9700 3400
-F 0 "R2" H 9770 3446 50  0000 L CNN
-F 1 "10K" H 9770 3355 50  0000 L CNN
-F 2 "Resistor_SMD:R_0805_2012Metric_Pad1.20x1.40mm_HandSolder" V 9630 3400 50  0001 C CNN
-F 3 "~" H 9700 3400 50  0001 C CNN
-	1    9700 3400
+P 9700 3540
+F 0 "R2" H 9770 3586 50  0000 L CNN
+F 1 "10K" H 9770 3495 50  0000 L CNN
+F 2 "Resistor_SMD:R_0805_2012Metric_Pad1.20x1.40mm_HandSolder" V 9630 3540 50  0001 C CNN
+F 3 "~" H 9700 3540 50  0001 C CNN
+	1    9700 3540
 	1    0    0    -1
 $EndComp
@@
 	9200 3400 9200 3800
 Wire Wire Line
-	9700 3550 9700 3800
-Wire Wire Line
-	9700 3250 9200 3250
-Wire Wire Line
-	9200 3250 9200 3400
+	9700 3690 9700 3800
 Connection ~ 9200 3400
 $Comp
@@
 	1    0    0    -1
 $EndComp
-Wire Wire Line
-	9200 2700 9200 3250
-Connection ~ 9200 3250
 Wire Wire Line
 	10150 2700 10150 3800
@@
 Wire Wire Line
 	3050 4450 3000 4450
+Text Notes 8100 7640 0    50   ~ 0
+11/22/2020
+Text Notes 7020 6660 0    50   ~ 0
+ATSAMD21E18BA-A based clone of adafruit's trinket m0, designed for EE101
+Text Notes 7330 7500 0    50   ~ 0
+tinyb0x
+Wire Wire Line
+	9200 2700 9200 2990
+Wire Wire Line
+	9700 3390 9700 2990
+Wire Wire Line
+	9700 2990 9200 2990
+Connection ~ 9200 2990
+Wire Wire Line
+	9200 2990 9200 3400
+$Comp
+L Connector_Generic:Conn_01x08 J2
+U 1 1 5FBB6050
+P 6740 1240
+F 0 "J2" V 6704 752 50  0000 R CNN
+F 1 "Conn_01x08" V 6613 752 50  0000 R CNN
+F 2 "Connector_PinHeader_2.54mm:PinHeader_1x08_P2.54mm_Vertical" H 6740 1240 50  0001 C CNN
+F 3 "~" H 6740 1240 50  0001 C CNN
+	1    6740 1240
+	0    -1   -1   0
+$EndComp
+Text GLabel 7140 1580 3    50   Input ~ 0
+D5_A5
+Text GLabel 7040 1580 3    50   Input ~ 0
+D4_A2
+Text GLabel 6940 1570 3    50   Input ~ 0
+D3_A3
+Text GLabel 6840 1570 3    50   Input ~ 0
+D2_A1
+Text GLabel 6740 1570 3    50   Input ~ 0
+D1_A0
+Text GLabel 6640 1560 3    50   Input ~ 0
+D0_A4
+Text GLabel 6540 1560 3    50   Input ~ 0
+3V3
+Text GLabel 6440 1550 3    50   Input ~ 0
+GND
+Wire Wire Line
+	6440 1550 6440 1440
+Wire Wire Line
+	6540 1440 6540 1560
+Wire Wire Line
+	6640 1440 6640 1560
+Wire Wire Line
+	6740 1440 6740 1570
+Wire Wire Line
+	6840 1440 6840 1570
+Wire Wire Line
+	6940 1440 6940 1570
+Wire Wire Line
+	7040 1440 7040 1580
+Wire Wire Line
+	7140 1440 7140 1580
 $EndSCHEMATC

Commit message: Add files via upload
Changed lines of the file:
@@
 U 1 1 5FAD07FB
 P 3150 5900
-F 0 "SW1" H 3150 6167 50  0000 C CNN
-F 1 "SW_DIP_x01" H 3150 6076 50  0000 C CNN
+F 0 "SW1" H 3220 6050 50  0000 C CNN
+F 1 "SW_DIP_x01" H 3170 5740 50  0000 C CNN
 F 2 "Button_Switch_SMD:SW_SPST_CK_RS282G05A3" H 3150 5900 50  0001 C CNN
 F 3 "~" H 3150 5900 50  0001 C CNN
@@
 U 1 1 5FAD41B4
 P 2950 2350
-F 0 "D1" H 2750 2800 50  0000 C CNN
-F 1 "APA102" H 2750 2700 50  0000 C CNN
+F 0 "D1" H 2790 2590 50  0000 C CNN
+F 1 "APA102" H 2790 2100 50  0000 C CNN
 F 2 "LED_SMD:LED_RGB_5050-6" H 3000 2050 50  0001 L TNN
 F 3 "http://www.led-color.com/upload/201506/APA102%20LED.pdf" H 3050 1975 50  0001 L TNN
@@
 U 1 1 5FAD9937
 P 2700 4650
-F 0 "J1" H 2757 5117 50  0000 C CNN
-F 1 "USB_B_Micro" H 2757 5026 50  0000 C CNN
+F 0 "J1" H 2870 4990 50  0000 C CNN
+F 1 "USB_B_Micro" H 2960 4310 50  0000 C CNN
 F 2 "Connector_USB:USB_Micro-B_Molex_47346-0001" H 2850 4600 50  0001 C CNN
 F 3 "~" H 2850 4600 50  0001 C CNN
@@
 U 1 1 5FBD726E
 P 4550 3850
-F 0 "U1" H 5180 3896 50  0000 L CNN
-F 1 "ATSAMD21E18A-A" H 5180 3805 50  0000 L CNN
+F 0 "U1" H 5050 5690 50  0000 L CNN
+F 1 "ATSAMD21E18A-A" H 4590 2000 50  0000 L CNN
 F 2 "Package_QFP:TQFP-32_7x7mm_P0.8mm" H 5450 2000 50  0001 C CNN
 F 3 "http://ww1.microchip.com/downloads/en/DeviceDoc/SAM_D21_DA1_Family_Data%20Sheet_DS40001882E.pdf" H 4550 3850 50  0001 C CNN
